File: kicad/oled - v0.9/Adafruit 128x64 Mono OLED PCB v2.sch (KiCad schematic (older format))
At the start: 53 parts, among them SW1 SW_Reed, SW2 SW_Reed, SW3 SW_Push, SW4 SW_Push, SW5 SW_Push, SW6 SW_Reed, U1 UG-2864HSWEG01

Commit message: Adicionando footprints.
Parts:
- removed BT3: Battery_Cell, symbol Device:Battery_Cell
- removed SJ1: -, Adafruit 128x64 Mono OLED PCB v2:SOLDERJUMPER_REFLOW_NOPASTE, symbol Adafruit_128x64_Mono_OLED_PCB_v2-eagle-import:SOLDERJUMPERREFLOW_NOPASTE
- removed U1: UG-2864HSWEG01, Adafruit 128x64 Mono OLED PCB v2:UG-2864HSWEG01_0.96IN_WRAPAROUND, symbol Adafruit_128x64_Mono_OLED_PCB_v2-eagle-import:DISP_OLED_UG-2864HSWEG010.96"
- BT1, BT2: footprint (none) -> Battery:Battery_Panasonic_CR2032-VS1N_Vertical_CircularHoles
- C10, C11, C12, C13, C2, C3, C4, C6, C8, C9: renamed from C?; footprint (none) -> Capacitor_SMD:C_0402_1005Metric
- C5: renamed from C?; value 100nF -> 4.7uF; footprint (none) -> Capacitor_SMD:C_0402_1005Metric
- C7: renamed from C?; value 1mF -> 1.0uF; footprint (none) -> Capacitor_SMD:C_0402_1005Metric
- L1, L2: renamed from L?; footprint (none) -> Inductor_SMD:L_0402_1005Metric
- L3: footprint (none) -> Inductor_SMD:L_0402_1005Metric
- R1, R10, R11, R12, R13, R14, R15, R16, R2, R3, R4, R5, R8, R9: footprint (none) -> Resistor_SMD:R_0402_1005Metric
- gave numbers to parts that had none: 3
Connections:
- net ButtonLeft: now also U1.7 (P0.05/AIN3)
- net ButtonRight: now also U1.6 (P0.04/AIN2)
- net CLK-I2C: now also U1.9 (P0.07); no longer U1.25 (SWDCLK)
- net LDR1A: now also U1.5 (P0.03/AIN1); no longer U1.10 (P0.08)
- net LDR1B: now also U1.4 (P0.02/AIN0); no longer U1.9 (P0.07)
- net CS-I2C: now reaches U1.11 (P0.09)
- net DATA-I2C: now reaches U1.8 (P0.06)
- net SDA-I2C: no longer names the net of U1.26 (SWDIO)
- new net SA0-I2C: U1.10 (P0.08)
- no-connect marks 39 -> 14
Other:
- note removed: "Bateria\nLCD"
- note removed: "Close for"
- note removed: "I2C"
- note removed: "OLED Display 128x64\nSSD1306"
- moved on the sheet: BT1, BT2, L1, L2

Commit message: Atualizando periféricos. Escolhendo footprints.
Parts:
- added AE1: Antenna, symbol Device:Antenna
- added C14: 2.2 pF, Capacitor_SMD:C_0402_1005Metric, symbol Device:C_Small
- added L4: 15nH, Inductor_SMD:L_0402_1005Metric, symbol Device:L_Small
- added L5: 3.9nH, Inductor_SMD:L_0402_1005Metric, symbol Device:L_Small
Connections:
- net GNDREF: now also L4.1
- net ANT: now reaches L3.2
- net ANT: now also C14.1
- new net: C14.2, L4.2, L5.1
- new net: AE1.1 (A), L5.2
Other:
- moved on the sheet: C9, L3
Changed lines of the file:
@@
 L Device:L_Small L3
 U 1 1 5E06A575
-P 5150 4365
-F 0 "L3" V 5208 4371 50  0000 L CNN
-F 1 "3.9nH" V 5080 4265 50  0000 L CNN
-F 2 "Inductor_SMD:L_0402_1005Metric" H 5150 4365 50  0001 C CNN
-F 3 "~" H 5150 4365 50  0001 C CNN
-	1    5150 4365
+P 4945 4365
+F 0 "L3" V 5003 4371 50  0000 L CNN
+F 1 "3.9nH" V 4875 4265 50  0000 L CNN
+F 2 "Inductor_SMD:L_0402_1005Metric" H 4945 4365 50  0001 C CNN
+F 3 "~" H 4945 4365 50  0001 C CNN
+	1    4945 4365
 	0    -1   -1   0
 $EndComp
@@
 L Device:C_Small C9
 U 1 1 5E43B6A7
-P 4900 4590
-F 0 "C9" H 4992 4636 50  0000 L CNN
-F 1 "0.8pF" H 4992 4545 50  0000 L CNN
-F 2 "Capacitor_SMD:C_0402_1005Metric" H 4900 4590 50  0001 C CNN
-F 3 "~" H 4900 4590 50  0001 C CNN
-	1    4900 4590
+P 4695 4590
+F 0 "C9" H 4787 4636 50  0000 L CNN
+F 1 "0.8pF" H 4787 4545 50  0000 L CNN
+F 2 "Capacitor_SMD:C_0402_1005Metric" H 4695 4590 50  0001 C CNN
+F 3 "~" H 4695 4590 50  0001 C CNN
+	1    4695 4590
 	1    0    0    -1
 $EndComp
 Wire Wire Line
-	4900 4490 4900 4365
+	4695 4490 4695 4365
 Wire Wire Line
-	4090 4365 4900 4365
-Connection ~ 4900 4365
-Wire Wire Line
-	4900 4365 5050 4365
+	4695 4365 4845 4365
 $Comp
 L power:GNDREF #PWR0112
 U 1 1 5E461BD7
-P 4900 4735
-F 0 "#PWR0112" H 4900 4485 50  0001 C CNN
-F 1 "GNDREF" H 4905 4562 50  0000 C CNN
-F 2 "" H 4900 4735 50  0001 C CNN
-F 3 "" H 4900 4735 50  0001 C CNN
-	1    4900 4735
+P 4695 4760
+F 0 "#PWR0112" H 4695 4510 50  0001 C CNN
+F 1 "GNDREF" H 4700 4587 50  0000 C CNN
+F 2 "" H 4695 4760 50  0001 C CNN
+F 3 "" H 4695 4760 50  0001 C CNN
+	1    4695 4760
 	1    0    0    -1
 $EndComp
 Wire Wire Line
-	4900 4735 4900 4710
-Wire Wire Line
-	4900 4710 4795 4710
-Wire Wire Line
-	4795 4710 4795 4265
-Wire Wire Line
-	4795 4265 4090 4265
-Connection ~ 4900 4710
-Wire Wire Line
-	4900 4710 4900 4690
-Wire Wire Line
-	5250 4365 5370 4365
+	5045 4365 5165 4365
 NoConn ~ 2890 3215
 NoConn ~ 2990 3215
@@
 Wire Wire Line
 	2590 1790 2980 1790
+Text GLabel 5165 4365 2    50   Input ~ 0
+ANT
+Wire Wire Line
+	4590 4265 4090 4265
+Wire Wire Line
+	4695 4365 4090 4365
+Connection ~ 4695 4365
+Wire Wire Line
+	4695 4690 4695 4725
+Wire Wire Line
+	4590 4265 4590 4725
+Wire Wire Line
+	4590 4725 4695 4725
+Connection ~ 4695 4725
+Wire Wire Line
+	4695 4725 4695 4760
+Text GLabel 4180 5600 0    50   Input ~ 0
+ANT
+$Comp
+L Device:C_Small C14
+U 1 1 5E360BE4
+P 4360 5600
+F 0 "C14" V 4462 5546 50  0000 L CNN
+F 1 "2.2 pF" V 4242 5495 50  0000 L CNN
+F 2 "Capacitor_SMD:C_0402_1005Metric" H 4360 5600 50  0001 C CNN
+F 3 "~" H 4360 5600 50  0001 C CNN
+	1    4360 5600
+	0    -1   -1   0
+$EndComp
+Wire Wire Line
+	4180 5600 4260 5600
+$Comp
+L Device:L_Small L5
+U 1 1 5E373FAB
+P 4975 5600
+F 0 "L5" V 5033 5606 50  0000 L CNN
+F 1 "3.9nH" V 4905 5500 50  0000 L CNN
+F 2 "Inductor_SMD:L_0402_1005Metric" H 4975 5600 50  0001 C CNN
+F 3 "~" H 4975 5600 50  0001 C CNN
+	1    4975 5600
+	0    -1   -1   0
+$EndComp
+$Comp
+L Device:L_Small L4
+U 1 1 5E382262
+P 4720 5785
+F 0 "L4" H 4768 5831 50  0000 L CNN
+F 1 "15nH" H 4768 5740 50  0000 L CNN
+F 2 "Inductor_SMD:L_0402_1005Metric" H 4720 5785 50  0001 C CNN
+F 3 "~" H 4720 5785 50  0001 C CNN
+	1    4720 5785
+	-1   0    0    1
+$EndComp
+Wire Wire Line
+	4460 5600 4720 5600
+Wire Wire Line
+	4720 5685 4720 5600
+Connection ~ 4720 5600
+Wire Wire Line
+	4720 5600 4875 5600
+Wire Wire Line
+	5075 5600 5175 5600
+Wire Wire Line
+	5175 5600 5175 5545
+$Comp
+L Device:Antenna AE1
+U 1 1 5E3B47C8
+P 5175 5345
+F 0 "AE1" H 5255 5334 50  0000 L CNN
+F 1 "Antenna" H 5255 5243 50  0000 L CNN
+F 2 "" H 5175 5345 50  0001 C CNN
+F 3 "~" H 5175 5345 50  0001 C CNN
+	1    5175 5345
+	1    0    0    -1
+$EndComp
+$Comp
+L power:GNDREF #PWR0113
+U 1 1 5E3BD3CB
+P 4720 5995
+F 0 "#PWR0113" H 4720 5745 50  0001 C CNN
+F 1 "GNDREF" H 4725 5822 50  0000 C CNN
+F 2 "" H 4720 5995 50  0001 C CNN
+F 3 "" H 4720 5995 50  0001 C CNN
+	1    4720 5995
+	1    0    0    -1
+$EndComp
+Wire Wire Line
+	4720 5995 4720 5885
 $EndSCHEMATC
